File: kicad/Mac DB15 to VGA TH v1.0.kicad_pcb (KiCad board)
At the start: 2 copper layers, 45.3 x 39.6 mm, 12 parts, among them J1 Mac_DB15_Male_MountingHoles, J2 VGA_DB15_Female_HighDensity_M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

Commit message: Add files via upload
Parts:
- added mrgasslogo: LOGO, project:mrgasslogo, B.Cu at (124.0, 104.5)
- SWA1, SWB1: footprint project:SW_DIP_SPSTx08_Slide_9.78x22.5mm_W7.62mm_P2.54mm -> Connector_PinHeader_2.54mm:PinHeader_2x08_P2.54mm_Vertical
- moved LOGOX 29.7 mm to (103.2, 93.5), turned to 90 degrees
- moved D3 18.7 mm to (114.2, 118.8), turned to 0 degrees
- moved D2 16.6 mm to (126.4, 122.5), turned to 0 degrees
- moved D6 11.4 mm to (134.1, 91.2), turned to 180 degrees
- moved D1 8.95 mm to (121.8, 122.5), turned to 180 degrees
- moved D5 7.93 mm to (126.4, 87.2), turned to 0 degrees
- moved D4 4.45 mm to (134.1, 118.8), turned to 180 degrees
- moved SWA1 3.17 mm to (118.8, 113.4)
- moved SWB1 3.12 mm to (131.0, 113.4)
- renumbered G*** to LOGO, G*** to LOGOX
Connections:
- SWA1 pad 10: Net-(SWA1-Pad10) -> (no net)
- SWA1 pad 11: Net-(SWA1-Pad11) -> (no net)
- SWA1 pad 6: Net-(SWA1-Pad6) -> (no net)
- SWA1 pad 7: Net-(SWA1-Pad7) -> (no net)
- SWA1 pad 8: Net-(SWA1-Pad8) -> (no net)
- SWA1 pad 9: Net-(SWA1-Pad9) -> (no net)
Routing:
- net /S1-1: track 24.0 -> 49.7 mm
- net /G: track 50.7 -> 32.6 mm
- net /GND: track 22.9 -> 7.20 mm, vias 50 -> 0
- net /S2-1: track 46.7 -> 59.7 mm, vias 2 -> 0
- net /D6: track 3.07 -> 13.4 mm
- net /HS: track 52.0 -> 41.6 mm, vias 2 -> 0
- net /R: track 42.2 -> 31.9 mm
- net /D5: track 5.71 -> 14.9 mm
- net /D2: track 21.9 -> 13.4 mm, vias 2 -> 0
- net /S0-1: track 60.1 -> 53.6 mm, vias 6 -> 0
- net /VS-2: track 38.8 -> 32.3 mm
- net /D1: track 20.4 -> 14.8 mm
- net /B: track 49.9 -> 53.8 mm, vias 2 -> 0
- net /HS-CS: track 21.1 -> 23.2 mm, vias 2 -> 0
- net /CS: track 18.6 -> 20.4 mm
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Other:
- net class Default removed
- board text added: "2022/08/17"
- board text added: "Customized for pin headers by"
- board text added: "Install 1N4148 diodes"
- board text added: "JLCJLCJLCJLC"
- board text added: "Sony MacView / UniMac 82D"
- board text added: "https://github.com/MrGasS"
- board text removed: "2021/11/18"
